Commit message: Added kuka example for BT testing

File: examples/youbot/robots/youbot.urdf.xacro (robot description, xacro)
@@ -30,5 +30,5 @@
 <!-- foot for arm-->
   <xacro:youbot_base name="base"/>
-  <!-- <xacro:youbot_plate name="plate" parent="base_link">
+  <xacro:youbot_plate name="plate" parent="base_link">
     <origin xyz="-0.159 0 0.046" rpy="0 0 0" />
   </xacro:youbot_plate>
@@ -38,4 +38,4 @@
   <xacro:youbot_gripper name="gripper" parent="arm_link_5">
     <origin xyz="0 0 0" rpy="0 0 0" />
-  </xacro:youbot_gripper> -->
+  </xacro:youbot_gripper>
 </robot>

File: examples/youbot/urdf/sensors/asus_xtion_camera.urdf.xacro (robot description, xacro)
@@ -28,5 +28,5 @@
         <origin xyz="0.01 0 0" rpy="${M_PI/2} 0 ${M_PI/2}" />
         <geometry>
-           <mesh filename="package://youbot_description/meshes/sensors/asus_xtion_pro_live_base.dae" scale="0.0004 0.0007 0.001"/>
+           <mesh filename="package://examples/youbot/meshes/sensors/asus_xtion_pro_live_base.dae" scale="0.0004 0.0007 0.001"/>
         </geometry>
         <material name="Black" />
@@ -35,5 +35,5 @@
         <origin xyz="0.01 0 0" rpy="${M_PI/2} 0 ${M_PI/2}" />
         <geometry>
-           <mesh filename="package://youbot_description/meshes/sensors/asus_xtion_pro_live_base.dae" scale="0.0004 0.0007 0.001"/>
+           <mesh filename="package://examples/youbot/meshes/sensors/asus_xtion_pro_live_base.dae" scale="0.0004 0.0007 0.001"/>
         </geometry>
       </collision >
@@ -81,5 +81,5 @@
         <origin xyz="0.02 -0.03 0" rpy="${M_PI/2} 0 ${M_PI/2}" />
         <geometry>
-          <mesh filename="package://youbot_description/meshes/sensors/asus_xtion_pro_live_camera.dae" scale="0.001 0.001 0.001"/>
+          <mesh filename="package://examples/youbot/meshes/sensors/asus_xtion_pro_live_camera.dae" scale="0.001 0.001 0.001"/>
         </geometry>
         <material name="Black" />
@@ -88,5 +88,5 @@
         <origin xyz="0.02 -0.03 0" rpy="${M_PI/2} 0 ${M_PI/2}" />
         <geometry>
-           <mesh filename="package://youbot_description/meshes/sensors/asus_xtion_pro_live_camera.dae" scale="0.001 0.001 0.001"/>
+           <mesh filename="package://examples/youbot/meshes/sensors/asus_xtion_pro_live_camera.dae" scale="0.001 0.001 0.001"/>
         </geometry>
       </collision >

File: examples/youbot/urdf/sensors/hokuyo_urg04_laser.urdf.xacro (robot description, xacro)
@@ -21,5 +21,5 @@
       	<origin xyz="0 0 0" rpy="0 0 0" />
 	<geometry>
-		<mesh filename="package://youbot_description/meshes/sensors/hokuyo.dae" />
+		<mesh filename="package://examples/youbot/meshes/sensors/hokuyo.dae" />
 	</geometry>
 	<material name="DarkGrey" />
@@ -28,5 +28,5 @@
 		<origin xyz="0 0 0" rpy="0 0 0" />
 		<geometry>
-			<mesh filename="package://youbot_description/meshes/sensors/hokuyo_convex.dae" />
+			<mesh filename="package://examples/youbot/meshes/sensors/hokuyo_convex.dae" />
 		</geometry>
 	</collision>

File: examples/youbot/urdf/sensors/kinect_camera.urdf.xacro (robot description, xacro)
@@ -22,5 +22,5 @@
       <origin xyz="0.0 0.0 0.0" rpy="0 0 0" />
       <geometry>
-       <mesh filename="package://youbot_description/meshes/sensors/kinect.dae"/>
+       <mesh filename="package://examples/youbot/meshes/sensors/kinect.dae"/>
       </geometry>
     </visual>
@@ -28,5 +28,5 @@
       <origin xyz="0.0 0.0 0.0" rpy="0 0 0" />
       <geometry>
-        <mesh filename="package://youbot_description/meshes/sensors/kinect.dae"/>
+        <mesh filename="package://examples/youbot/meshes/sensors/kinect.dae"/>
       </geometry>
     </collision>

File: examples/youbot/urdf/sensors/microsoft_lifecam.urdf.xacro (robot description, xacro)
@@ -22,5 +22,5 @@
       <origin xyz="-0.04 -0.0035 -0.031" rpy="${M_PI/2} 0 ${M_PI/2}" />
       <geometry>
-       <mesh filename="package://youbot_description/meshes/sensors/microsoft_lifecam.dae" scale="0.001 0.001 0.001"/>
+       <mesh filename="package://examples/youbot/meshes/sensors/microsoft_lifecam.dae" scale="0.001 0.001 0.001"/>
       </geometry>
     </visual>
@@ -28,5 +28,5 @@
       <origin xyz="-0.04 -0.0035 -0.031" rpy="${M_PI/2} 0 ${M_PI/2}" />
       <geometry>
-        <mesh filename="package://youbot_description/meshes/sensors/microsoft_lifecam.dae" scale="0.001 0.001 0.001"/>
+        <mesh filename="package://examples/youbot/meshes/sensors/microsoft_lifecam.dae" scale="0.001 0.001 0.001"/>
       </geometry>
     </collision>

File: examples/youbot/urdf/youbot_arm/arm.urdf.xacro (robot description, xacro)
@@ -24,5 +24,5 @@
 				<origin xyz="0 0 0" rpy="0 0 0" />
 				<geometry>
-					<mesh filename="package://youbot_description/meshes/youbot_arm/arm0.dae" />
+					<mesh filename="package://examples/youbot/meshes/youbot_arm/arm0.dae" />
 				</geometry>
 				<material name="DarkGrey" />
@@ -32,5 +32,5 @@
 				<origin xyz="0 0 0" rpy="0 0 0"/>
 				<geometry>
-					<mesh filename="package://youbot_description/meshes/youbot_arm/arm0_convex.dae" />
+					<mesh filename="package://examples/youbot/meshes/youbot_arm/arm0_convex.dae" />
 					<!--<cylinder length="0.078" radius="0.093"/>-->
 				</geometry>
@@ -63,5 +63,5 @@
 				<origin xyz="0 0 0" rpy="0 0 0" />
 				<geometry>
-					<mesh filename="package://youbot_description/meshes/youbot_arm/arm1.dae" />
+					<mesh filename="package://examples/youbot/meshes/youbot_arm/arm1.dae" />
 				</geometry>
 				<!--<material name="Orange" />-->
@@ -71,5 +71,5 @@
 				<origin xyz="0 0 0" rpy="0 0 0" />
 				<geometry>
-					<mesh filename="package://youbot_description/meshes/youbot_arm/arm1_convex.dae" />
+					<mesh filename="package://examples/youbot/meshes/youbot_arm/arm1_convex.dae" />
 					<!--<cylinder length="0.102" radius="0.080"/>-->
 				</geometry>
@@ -95,5 +95,5 @@
 			<origin xyz="0 -0.032 0.078" rpy="0 0 0" />
 				<geometry>
-					<mesh filename="package://youbot_description/meshes/youbot_arm/arm2.dae" />
+					<mesh filename="package://examples/youbot/meshes/youbot_arm/arm2.dae" />
 				</geometry>
 				<material name="Orange" />
@@ -103,5 +103,5 @@
 				<origin xyz="0 -0.032 0.078" rpy="0 0 0" />
 				<geometry>
-					<mesh filename="package://youbot_description/meshes/youbot_arm/arm2_convex.dae" />
+					<mesh filename="package://examples/youbot/meshes/youbot_arm/arm2_convex.dae" />
 					<!--<box size="0.074 0.082 0.222"/>-->
 				</geometry>
@@ -135,5 +135,5 @@
 				<origin xyz="0.000 0.028 0.079" rpy="0 0 0" />
 				<geometry>
-					<mesh filename="package://youbot_description/meshes/youbot_arm/arm3.dae" />
+					<mesh filename="package://examples/youbot/meshes/youbot_arm/arm3.dae" />
 				</geometry>
 				<material name="Orange" />
@@ -143,5 +143,5 @@
 				<origin xyz="0.000 0.028 0.079" rpy="0 0 0" />
 				<geometry>
-					<mesh filename="package://youbot_description/meshes/youbot_arm/arm3_convex.dae" />
+					<mesh filename="package://examples/youbot/meshes/youbot_arm/arm3_convex.dae" />
 					<!--<box size="0.064 0.054 0.192"/>-->
 				</geometry>
@@ -167,5 +167,5 @@
 				<origin xyz="0 -0.010 0.029" rpy="0 0 0"/>
 				<geometry>
-					<mesh filename="package://youbot_description/meshes/youbot_arm/arm4.dae" />
+					<mesh filename="package://examples/youbot/meshes/youbot_arm/arm4.dae" />
 				</geometry>
 				<material name="Orange" />
@@ -175,5 +175,5 @@
 				<origin xyz="0 -0.010 0.029" rpy="0 0 0"/>
 				<geometry>
-					<mesh filename="package://youbot_description/meshes/youbot_arm/arm4_convex.dae" />
+					<mesh filename="package://examples/youbot/meshes/youbot_arm/arm4_convex.dae" />
 					<!--<box size="0.058 0.100 0.118"/>-->
 				</geometry>
@@ -199,5 +199,5 @@
 				<origin xyz="0.003 0 -0.034" rpy="0 0 0" />
 				<geometry>
-					<mesh filename="package://youbot_description/meshes/youbot_arm/arm5.dae" />
+					<mesh filename="package://examples/youbot/meshes/youbot_arm/arm5.dae" />
 				</geometry>
 				<material name="DarkGrey" />
@@ -206,5 +206,5 @@
 				<origin xyz="0.003 0 -0.034" rpy="0 0 0" />
 				<geometry>
-					<mesh filename="package://youbot_description/meshes/youbot_arm/arm5_convex.dae" />
+					<mesh filename="package://examples/youbot/meshes/youbot_arm/arm5_convex.dae" />
 					<!--<box size="0.054 0.096 0.030"/>-->
 				</geometry>

File: examples/youbot/urdf/youbot_base/base.urdf.xacro (robot description, xacro)
@@ -70,5 +70,5 @@
         			<origin xyz="0 0 0" rpy="0 0 0" />
         			<geometry>
-          				<mesh filename="package://youbot_description/meshes/youbot_base/base.dae"/>
+          				<mesh filename="package://examples/youbot/meshes/youbot_base/base.dae"/>
         			</geometry>
         			<material name="DarkGrey"/>
@@ -78,5 +78,5 @@
         			<geometry>
           				<!--<box size="${base_size_x} ${base_size_y} ${base_size_z}" />-->
-					<mesh filename="package://youbot_description/meshes/youbot_base/base_convex.dae"/>
+					<mesh filename="package://examples/youbot/meshes/youbot_base/base_convex.dae"/>
 	       			</geometry>
       			</collision>
@@ -122,5 +122,5 @@
       			<visual>
         			<origin xyz="0 0 0" rpy="0 0 0" />
-					<!--<mesh filename="package://youbot_description/meshes/youbot_base/youbot_wheel.stl" />-->
+					<!--<mesh filename="package://examples/youbot/meshes/youbot_base/youbot_wheel.stl" />-->
 				<geometry>
 					<sphere radius="${wheel_radius}"/>
@@ -172,5 +172,5 @@
         			<origin xyz="0 0 0" rpy="0 0 0" />
 				<geometry>
-          				<!--<mesh filename="package://youbot_description/meshes/youbot_base/youbot_wheel.stl" />-->
+          				<!--<mesh filename="package://examples/youbot/meshes/youbot_base/youbot_wheel.stl" />-->
 					<sphere radius="${wheel_radius}"/>
         			</geometry>
@@ -222,5 +222,5 @@
         			<origin xyz="0 0 0" rpy="0 0 0" />
 				<geometry>
-          				<!--<mesh filename="package://youbot_description/meshes/youbot_base/youbot_wheel.stl" />-->
+          				<!--<mesh filename="package://examples/youbot/meshes/youbot_base/youbot_wheel.stl" />-->
 					<sphere radius="${wheel_radius}"/>
         			</geometry>
@@ -271,5 +271,5 @@
         			<origin xyz="0 0 0" rpy="0 0 0" />
 				<geometry>
-          				<!--<mesh filename="package://youbot_description/meshes/youbot_base/youbot_wheel.stl" />-->
+          				<!--<mesh filename="package://examples/youbot/meshes/youbot_base/youbot_wheel.stl" />-->
 					<sphere radius="${wheel_radius}"/>
         			</geometry>

File: examples/youbot/urdf/youbot_gripper/gripper.urdf.xacro (robot description, xacro)
@@ -23,5 +23,5 @@
 				<origin xyz="0 0 0" rpy="0 0 0" />
 				<geometry>
-					<mesh filename="package://youbot_description/meshes/youbot_gripper/palm.dae" />
+					<mesh filename="package://examples/youbot/meshes/youbot_gripper/palm.dae" />
 				</geometry>
 				<material name="Black" />
@@ -31,5 +31,5 @@
 				<geometry>
 					<!--<box size="0.050 0.094 0.054"/>-->
-					<mesh filename="package://youbot_description/meshes/youbot_gripper/palm_convex.dae" />
+					<mesh filename="package://examples/youbot/meshes/youbot_gripper/palm_convex.dae" />
 				</geometry>
 			</collision>
@@ -53,5 +53,5 @@
 				<origin xyz="0 0 0" rpy="0 0 0" />
 				<geometry>
-					<mesh filename="package://youbot_description/meshes/youbot_gripper/finger.dae" />
+					<mesh filename="package://examples/youbot/meshes/youbot_gripper/finger.dae" />
 				</geometry>
 				<material name="Black" />
@@ -61,5 +61,5 @@
 				<geometry>
 					<!--<box size="0.014 0.020 0.046"/>-->
-					<mesh filename="package://youbot_description/meshes/youbot_gripper/finger_convex.dae" />
+					<mesh filename="package://examples/youbot/meshes/youbot_gripper/finger_convex.dae" />
 				</geometry>
 			</collision>
@@ -83,5 +83,5 @@
 				<origin xyz="0 0 0" rpy="0 0 0" />
 				<geometry>
-					<mesh filename="package://youbot_description/meshes/youbot_gripper/finger.dae" />
+					<mesh filename="package://examples/youbot/meshes/youbot_gripper/finger.dae" />
 				</geometry>
 				<material name="Black" />
@@ -91,5 +91,5 @@
 				<geometry>
 					<!--<box size="0.014 0.020 0.046"/>-->
-					<mesh filename="package://youbot_description/meshes/youbot_gripper/finger_convex.dae" />
+					<mesh filename="package://examples/youbot/meshes/youbot_gripper/finger_convex.dae" />
 				</geometry>
 			</collision>

File: examples/youbot/urdf/youbot_plate/plate.urdf.xacro (robot description, xacro)
@@ -20,5 +20,5 @@
 				<origin xyz="0 0 0" rpy="0 0 0" />
 				<geometry>
-					<mesh filename="package://youbot_description/meshes/youbot_plate/plate.dae" />
+					<mesh filename="package://examples/youbot/meshes/youbot_plate/plate.dae" />
 				</geometry>
 				<material name="DarkGrey"/>
@@ -27,5 +27,5 @@
 				<origin xyz="0 0 0" rpy="0 0 0" />
 				<geometry>
-					<mesh filename="package://youbot_description/meshes/youbot_plate/plate_convex.dae" />
+					<mesh filename="package://examples/youbot/meshes/youbot_plate/plate_convex.dae" />
 				</geometry>
 			</collision>
